File: cad/mini_optron/mini_optron.sch (EAGLE design)
At the start: 10 parts

Commit message: Updated FSR circuit, c1 orient
Parts:
- R1: value 2.2k -> 33k
Connections:
- net CONN: now also FORCE_JP.1
- net VCC: no longer FORCE_JP.1
Changed lines of the file:
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@@
 <?xml version="1.0" encoding="utf-8"?>
 <!DOCTYPE eagle SYSTEM "eagle.dtd">
-<eagle version="9.6.1">
+<eagle version="9.3.1">
 <drawing>
 <settings>
@@
 </part>
 <part name="P+1" library="supply1" library_urn="urn:adsk.eagle:library:371" deviceset="VCC" device=""/>
-<part name="P+2" library="supply1" library_urn="urn:adsk.eagle:library:371" deviceset="VCC" device=""/>
 <part name="P+3" library="supply1" library_urn="urn:adsk.eagle:library:371" deviceset="VCC" device=""/>
 <part name="SUPPLY1" library="supply2" library_urn="urn:adsk.eagle:library:372" deviceset="GND" device=""/>
@@
 <part name="SOFT_POT_JP" library="pinhead" library_urn="urn:adsk.eagle:library:325" deviceset="PINHD-1X3" device="" package3d_urn="urn:adsk.eagle:package:22458/2"/>
 <part name="DOTSTAR_JP" library="pinhead" library_urn="urn:adsk.eagle:library:325" deviceset="PINHD-1X4" device="" package3d_urn="urn:adsk.eagle:package:22407/2"/>
-<part name="R1" library="SparkFun-Resistors" library_urn="urn:adsk.eagle:library:532" deviceset="RESISTOR" device="AXIAL-0.3" package3d_urn="urn:adsk.eagle:package:39658/1" value=" 2.2k">
+<part name="R1" library="SparkFun-Resistors" library_urn="urn:adsk.eagle:library:532" deviceset="RESISTOR" device="AXIAL-0.3" package3d_urn="urn:adsk.eagle:package:39658/1" value="33k">
 <attribute name="MF" value="VISHAY"/>
 <attribute name="MPN" value="CRCW060310K0FKEA"/>
@@
 <attribute name="VALUE" x="78.74" y="58.42" size="1.778" layer="96"/>
 </instance>
-<instance part="P+2" gate="VCC" x="30.48" y="58.42" smashed="yes" rot="R270">
-<attribute name="VALUE" x="30.48" y="58.42" size="1.778" layer="96"/>
-</instance>
 <instance part="P+3" gate="VCC" x="22.86" y="27.94" smashed="yes">
 <attribute name="VALUE" x="25.4" y="30.48" size="1.778" layer="96" rot="R180"/>
@@
 <wire x1="22.86" y1="22.86" x2="35.56" y2="22.86" width="0.1524" layer="91"/>
 </segment>
-<segment>
-<pinref part="P+2" gate="VCC" pin="VCC"/>
-<pinref part="FORCE_JP" gate="G$1" pin="1"/>
-<wire x1="27.94" y1="58.42" x2="20.32" y2="58.42" width="0.1524" layer="91"/>
-</segment>
 </net>
 <net name="N$4" class="0">
@@
 <wire x1="12.7" y1="63.5" x2="33.02" y2="63.5" width="0.1524" layer="91"/>
 <label x="33.02" y="71.12" size="1.778" layer="95" rot="R180" xref="yes"/>
-</segment>
-</net>
+<pinref part="FORCE_JP" gate="G$1" pin="1"/>
+<wire x1="33.02" y1="58.42" x2="20.32" y2="58.42" width="0.1524" layer="91"/>
+<wire x1="33.02" y1="58.42" x2="33.02" y2="63.5" width="0.1524" layer="91"/>
+</segment>
+</net>

Commit message: Add files via upload
Parts:
- removed R2: 10k, SparkFun-Resistors:RESISTORAXIAL-0.3
- R1: value 33k -> 10K
Connections:
- net N$1 renamed A0
- removed net CONN: FORCE_JP.1, JP1.2, MPU6050_JP.1, R2.1
- removed net N$10: JP2.12, MPU6050_JP.4
- removed net N$2: DOTSTAR_JP.2, JP1.11
- removed net N$3: R2.2, SOFT_POT_JP.1
- removed net N$4: JP1.6, SOFT_POT_JP.2
- removed net N$5: R3.2, SOFT_POT_JP.3
- removed net N$6: DOTSTAR_JP.3, JP1.12
- removed net N$9: JP2.11, MPU6050_JP.3
- removed net VCC: C1.1, DOTSTAR_JP.1, JP2.3
- new net 3V: FORCE_JP.1, JP1.2, MPU6050_JP.3, SOFT_POT_JP.1
- new net 5V: C1.1, DOTSTAR_JP.3, JP2.3
- new net A1: JP1.6, R3.2, SOFT_POT_JP.3
- new net MOSI: DOTSTAR_JP.2, JP1.12
- new net SCK: DOTSTAR_JP.1, JP1.11
- new net SCL: JP2.11, MPU6050_JP.1
- new net SDA: JP2.12, MPU6050_JP.2
- net GND: now also MPU6050_JP.4, SOFT_POT_JP.2; no longer MPU6050_JP.2
Other:
- moved on the sheet: C1, DOTSTAR_JP, FORCE_JP, MPU6050_JP, R1, R3, SOFT_POT_JP
